Commit message: Update gen3_lite_macro_modified.xacro

File: kortex_description/arms/gen3_lite/6dof/urdf/gen3_lite_macro_modified.xacro (robot description, xacro)
@@ -3,5 +3,4 @@
   <!-- Propagate last link name information because it is the gripper's parent link -->
   <xacro:property name="last_arm_link" value="dummy_link"/>
-  <xacro:macro name="load_arm" params="parent:='' dof vision prefix *origin">
     <link name="table_link">
       <visual>
@@ -19,4 +18,26 @@
       <origin xyz="0.25 0 -0.0627" rpy="0 0 1.57"/>
     </joint>
+    <link name="cup_link">
+      <visual>
+        <geometry>
+          <cylinder length="0.125" radius="0.0425"/>
+        </geometry>
+        <material name="white">
+          <color rgba="1 1 1 1"/>
+        </material>
+      </visual>
+      <collision>
+        <origin xyz="0 0 0" rpy="0 0 0" />
+        <geometry>
+          <mesh filename="package://kortex_description/arms/gen3_lite/${dof}dof/meshes/base_link.STL" />
+        </geometry>
+      </collision>
+    </link>
+    <joint name="cup_joint" type="fixed">
+      <parent link="${prefix}end_effector_link"/>
+      <child link="cup_link"/>
+      <origin xyz="0.0 0 0.12" rpy="0 1.57 0"/>
+    </joint>
+  <xacro:macro name="load_arm" params="parent:='' dof vision prefix *origin">
     <link name="${prefix}base_link">
       <inertial>

Commit message: Added mug stl file and updated xarco file

File: kortex_description/arms/gen3_lite/6dof/urdf/gen3_lite_macro_modified.xacro (robot description, xacro)
@@ -21,5 +21,6 @@
       <visual>
         <geometry>
-          <cylinder length="0.125" radius="0.0425"/>
+          <!-- <cylinder length="0.125" radius="0.0425"/> -->
+          <mesh filename="package://kortex_description/arms/gen3_lite/${dof}dof/meshes/MugCylinder.stl" scale="0.01 0.01 0.01"/>
         </geometry>
         <material name="white">
@@ -30,5 +31,5 @@
         <origin xyz="0 0 0" rpy="0 0 0" />
         <geometry>
-          <mesh filename="package://kortex_description/arms/gen3_lite/${dof}dof/meshes/base_link.STL" />
+          <mesh filename="package://kortex_description/arms/gen3_lite/${dof}dof/meshes/MugCylinder.stl" scale="0.01 0.01 0.01"/>
         </geometry>
       </collision>
@@ -37,5 +38,5 @@
       <parent link="${prefix}end_effector_link"/>
       <child link="cup_link"/>
-      <origin xyz="0.0 0 0.12" rpy="0 1.57 0"/>
+      <origin xyz="0.0 0 0.12" rpy="-1.57 03.14 0"/>
     </joint>
   <xacro:macro name="load_arm" params="parent:='' dof vision prefix *origin">

Commit message: Update gen3_lite_macro_modified.xacro

File: kortex_description/arms/gen3_lite/6dof/urdf/gen3_lite_macro_modified.xacro (robot description, xacro)
@@ -40,4 +40,26 @@
       <origin xyz="0.0 0 0.12" rpy="-1.57 03.14 0"/>
     </joint>
+    <link name="cup_link2">
+      <visual>
+        <geometry>
+          <!-- <cylinder length="0.125" radius="0.0425"/> -->
+          <mesh filename="package://kortex_description/arms/gen3_lite/${dof}dof/meshes/MugCylinder.stl" scale="0.01 0.01 0.01"/>
+        </geometry>
+        <material name="white">
+          <color rgba="1 1 1 1"/>
+        </material>
+      </visual>
+      <collision>
+        <origin xyz="0 0 0" rpy="0 0 0" />
+        <geometry>
+          <mesh filename="package://kortex_description/arms/gen3_lite/${dof}dof/meshes/MugCylinder.stl" scale="0.01 0.01 0.01"/>
+        </geometry>
+      </collision>
+    </link>
+    <joint name="cup_joint2" type="fixed">
+      <parent link="table_link"/>
+      <child link="cup_link2"/>
+      <origin xyz="0.15 -0.23 0.0625" rpy="0 1.57 0"/>
+    </joint>
   <xacro:macro name="load_arm" params="parent:='' dof vision prefix *origin">
     <link name="${prefix}base_link">

Commit message: Update gen3_lite_macro_modified.xacro

File: kortex_description/arms/gen3_lite/6dof/urdf/gen3_lite_macro_modified.xacro (robot description, xacro)
@@ -31,5 +31,5 @@
         <origin xyz="0 0 0" rpy="0 0 0" />
         <geometry>
-          <mesh filename="package://kortex_description/arms/gen3_lite/${dof}dof/meshes/MugCylinder.stl" scale="0.01 0.01 0.01"/>
+          <mesh filename="package://kortex_description/arms/gen3_lite/${dof}dof/meshes/MugCylinder.stl" scale="0.001 0.001 0.001"/>
         </geometry>
       </collision>

Commit message: updated 3d models

File: kortex_description/arms/gen3_lite/6dof/urdf/gen3_lite_macro_modified.xacro (robot description, xacro)
@@ -40,26 +40,66 @@
       <origin xyz="0.0 0 0.12" rpy="-1.57 03.14 0"/>
     </joint>
-    <link name="target_cup0">
-      <visual>
-        <origin xyz="0 0 0" rpy="0 0 0" />
-        <geometry>
-          <!-- <cylinder length="0.125" radius="0.0425"/> -->
-          <mesh filename="package://kortex_description/arms/gen3_lite/${dof}dof/meshes/MugCylinder.stl" scale="0.01 0.01 0.01"/>
-        </geometry>
-        <material name="white">
-          <color rgba="1 1 1 1"/>
-        </material>
-      </visual>
-      <collision>
-        <origin xyz="0 0 0" rpy="0 0 0" />
-        <geometry>
-          <mesh filename="package://kortex_description/arms/gen3_lite/${dof}dof/meshes/MugCylinder.stl" scale="0.01 0.01 0.01"/>
-        </geometry>
-      </collision>
-    </link>
-    <joint name="cup_joint0" type="fixed">
-      <parent link="table_link"/>
-      <child link="target_cup0"/>
-      <origin xyz="0.15 -0.23 0.0625" rpy="0 1.57 0"/>
+    <link name="coffee_cup">
+      <visual>
+        <geometry>
+          <mesh filename="package://kortex_description/arms/gen3_lite/${dof}dof/meshes/papercup.stl" scale="1 1 1"/>
+        </geometry>
+        <material name="green">
+          <color rgba="0 1 0 1"/>
+        </material>
+      </visual>
+      <collision>
+        <origin xyz="0 0 0" rpy="0 0 0" />
+        <geometry>
+          <mesh filename="package://kortex_description/arms/gen3_lite/${dof}dof/meshes/papercup.stl" scale="0.001 0.001 0.001"/>
+        </geometry>
+      </collision>
+    </link>
+    <joint name="papercup_joint" type="fixed">
+      <parent link="${prefix}end_effector_link"/>
+      <child link="coffee_cup"/>
+      <origin xyz="0.0 0 0.12" rpy="-1.57 0 -1.57"/>
+    </joint>
+    <link name="soda_can">
+      <visual>
+        <geometry>
+          <mesh filename="package://kortex_description/arms/gen3_lite/${dof}dof/meshes/beverage_can.fbx" scale="0.01 0.01 0.01"/>
+        </geometry>
+        <material name="green">
+          <color rgba="0 1 0 1"/>
+        </material>
+      </visual>
+      <collision>
+        <origin xyz="0 0 0" rpy="0 0 0" />
+        <geometry>
+          <mesh filename="package://kortex_description/arms/gen3_lite/${dof}dof/meshes/beverage_can.fbx" scale="0.001 0.001 0.001"/>
+        </geometry>
+      </collision>
+    </link>
+    <joint name="sodacan_joint" type="fixed">
+      <parent link="${prefix}end_effector_link"/>
+      <child link="soda_can"/>
+      <origin xyz="-0.04 0.0 0.12" rpy="0 0 -1.57"/>
+    </joint>
+    <link name="water_bottle">
+      <visual>
+        <geometry>
+          <mesh filename="package://kortex_description/arms/gen3_lite/${dof}dof/meshes/water_bottle.stl" scale="1 1 1"/>
+        </geometry>
+        <material name="green">
+          <color rgba="0 1 0 1"/>
+        </material>
+      </visual>
+      <collision>
+        <origin xyz="0 0 0" rpy="0 0 0" />
+        <geometry>
+          <mesh filename="package://kortex_description/arms/gen3_lite/${dof}dof/meshes/water_bottle.stl" scale="0.001 0.001 0.001"/>
+        </geometry>
+      </collision>
+    </link>
+    <joint name="waterbottle_joint" type="fixed">
+      <parent link="${prefix}end_effector_link"/>
+      <child link="water_bottle"/>
+      <origin xyz="0.0 0.0 0.12" rpy="0 1.57 0"/>
     </joint>
     <link name="target_cup1">
@@ -84,50 +124,4 @@
       <parent link="table_link"/>
       <child link="target_cup1"/>
-      <origin xyz="0.0 -0.23 0.0625" rpy="0 1.57 0"/>
-    </joint>
-    <link name="target_cup34">
-      <visual>
-        <origin xyz="0 0 0" rpy="0 0 0" />
-        <geometry>
-          <!-- <cylinder length="0.125" radius="0.0425"/> -->
-          <mesh filename="package://kortex_description/arms/gen3_lite/${dof}dof/meshes/MugCylinder.stl" scale="0.01 0.01 0.01"/>
-        </geometry>
-        <material name="white">
-          <color rgba="1 1 1 1"/>
-        </material>
-      </visual>
-      <collision>
-        <origin xyz="0 0 0" rpy="0 0 0" />
-        <geometry>
-          <mesh filename="package://kortex_description/arms/gen3_lite/${dof}dof/meshes/MugCylinder.stl" scale="0.01 0.01 0.01"/>
-        </geometry>
-      </collision>
-    </link>
-    <joint name="cup_joint34" type="fixed">
-      <parent link="table_link"/>
-      <child link="target_cup34"/>
-      <origin xyz="0.15 -0.23 0.0625" rpy="0 0 0"/>
-    </joint>
-    <link name="target_cup2">
-      <visual>
-        <origin xyz="0 0 0" rpy="0 0 0" />
-        <geometry>
-          <!-- <cylinder length="0.125" radius="0.0425"/> -->
-          <mesh filename="package://kortex_description/arms/gen3_lite/${dof}dof/meshes/Can.stl" />
-        </geometry>
-        <material name="white">
-          <color rgba="1 1 1 1"/>
-        </material>
-      </visual>
-      <collision>
-        <origin xyz="0 0 0" rpy="0 0 0" />
-        <geometry>
-          <mesh filename="package://kortex_description/arms/gen3_lite/${dof}dof/meshes/Can.stl"/>
-        </geometry>
-      </collision>
-    </link>
-    <joint name="cup_joint3" type="fixed">
-      <parent link="table_link"/>
-      <child link="target_cup2"/>
       <origin xyz="0.0 -0.23 0.0625" rpy="0 1.57 0"/>
     </joint>

Commit message: updated pouring scene

File: kortex_description/arms/gen3_lite/6dof/urdf/gen3_lite_macro_modified.xacro (robot description, xacro)
@@ -82,8 +82,8 @@
       <origin xyz="-0.04 0.0 0.12" rpy="0 0 -1.57"/>
     </joint>
-    <link name="water_bottle">
-      <visual>
-        <geometry>
-          <mesh filename="package://kortex_description/arms/gen3_lite/${dof}dof/meshes/water_bottle.stl" scale="1 1 1"/>
+    <!-- <link name="beer_bottle">
+      <visual>
+        <geometry>
+          <mesh filename="package://kortex_description/arms/gen3_lite/${dof}dof/meshes/beer_bottle.stl" scale="0.001 0.001 0.001"/>
         </geometry>
         <material name="green">
@@ -94,5 +94,5 @@
         <origin xyz="0 0 0" rpy="0 0 0" />
         <geometry>
-          <mesh filename="package://kortex_description/arms/gen3_lite/${dof}dof/meshes/water_bottle.stl" scale="0.001 0.001 0.001"/>
+          <mesh filename="package://kortex_description/arms/gen3_lite/${dof}dof/meshes/beer_bottle.stl" scale="0.001 0.001 0.001"/>
         </geometry>
       </collision>
@@ -100,7 +100,7 @@
     <joint name="waterbottle_joint" type="fixed">
       <parent link="${prefix}end_effector_link"/>
-      <child link="water_bottle"/>
-      <origin xyz="0.0 0.0 0.12" rpy="0 1.57 0"/>
-    </joint>
+      <child link="beer_bottle"/>
+      <origin xyz="0.0 0.0 0.1" rpy="0 1.57 0"/>
+    </joint> -->
     <link name="target_cup1">
       <visual>

Commit message: Added  source models

File: kortex_description/arms/gen3_lite/6dof/urdf/gen3_lite_macro_modified.xacro (robot description, xacro)
@@ -18,96 +18,95 @@
       <origin xyz="0.25 0 -0.0627" rpy="0 0 1.57"/>
     </joint>
-    <link name="source_cup">
-      <visual>
+    <link name="10_Mug">
+      <visual>
+        <geometry>
+          <mesh filename="package://kortex_description/arms/gen3_lite/${dof}dof/meshes/10_mug.fbx" scale="1 1 1"/>
+        </geometry>
+        <material name="green">
+          <color rgba="0 1 0 1"/>
+        </material>
+      </visual>
+      <collision>
+        <origin xyz="0 0 0" rpy="0 0 0" />
+        <geometry>
+          <mesh filename="package://kortex_description/arms/gen3_lite/${dof}dof/meshes/10_mug.fbx" scale="0.001 0.001 0.001"/>
+        </geometry>
+      </collision>
+    </link>
+    <joint name="mug_joint" type="fixed">
+      <parent link="${prefix}end_effector_link"/>
+      <child link="10_Mug"/>
+      <origin xyz="0.0 0 0" rpy="0 0 0"/>
+    </joint>
+    <link name="09_PaperCup">
+      <visual>
+        <geometry>
+          <mesh filename="package://kortex_description/arms/gen3_lite/${dof}dof/meshes/09_Paper_cup.fbx" scale="1 1 1"/>
+        </geometry>
+        <material name="green">
+          <color rgba="0 1 0 1"/>
+        </material>
+      </visual>
+      <collision>
+        <origin xyz="0 0 0" rpy="0 0 0" />
+        <geometry>
+          <mesh filename="package://kortex_description/arms/gen3_lite/${dof}dof/meshes/09_Paper_cup.fbx" scale="0.001 0.001 0.001"/>
+        </geometry>
+      </collision>
+    </link>
+    <joint name="papercup_joint" type="fixed">
+      <parent link="${prefix}end_effector_link"/>
+      <child link="09_PaperCup"/>
+      <origin xyz="0.0 0 0" rpy="0 0 0"/>
+    </joint>
+    <link name="01_Can">
+      <visual>
+        <geometry>
+          <mesh filename="package://kortex_description/arms/gen3_lite/${dof}dof/meshes/01_Can.fbx" scale="1 1 1"/>
+        </geometry>
+        <material name="green">
+          <color rgba="0 1 0 1"/>
+        </material>
+      </visual>
+      <collision>
+        <origin xyz="0 0 0" rpy="0 0 0" />
+        <geometry>
+          <mesh filename="package://kortex_description/arms/gen3_lite/${dof}dof/meshes/01_Can.fbx" scale="0.001 0.001 0.001"/>
+        </geometry>
+      </collision>
+    </link>
+    <joint name="sodacan_joint" type="fixed">
+      <parent link="${prefix}end_effector_link"/>
+      <child link="01_Can"/>
+      <origin xyz="-0.0 0.0 0" rpy="0 0 0"/>
+    </joint>
+    <link name="07_Rootbeer">
+      <visual>
+        <geometry>
+          <mesh filename="package://kortex_description/arms/gen3_lite/${dof}dof/meshes/08_beerbottle.fbx"/>
+        </geometry>
+        <material name="green">
+          <color rgba="0 1 0 1"/>
+        </material>
+      </visual>
+      <collision>
+        <origin xyz="0 0 0" rpy="0 0 0" />
+        <geometry>
+          <mesh filename="package://kortex_description/arms/gen3_lite/${dof}dof/meshes/08_beerbottle.fbx" scale="0.001 0.001 0.001"/>
+        </geometry>
+      </collision>
+    </link>
+    <joint name="beer_bottle_joint" type="fixed">
+      <parent link="${prefix}end_effector_link"/>
+      <child link="07_Rootbeer"/>
+      <origin xyz="0.0 0.0 0.0" rpy="0 0 0"/>
+    </joint>
+    <link name="Target_Cup">
+      <visual>
+        <origin xyz="0 0 0" rpy="0 0 0" />
         <geometry>
           <!-- <cylinder length="0.125" radius="0.0425"/> -->
           <mesh filename="package://kortex_description/arms/gen3_lite/${dof}dof/meshes/MugCylinder.stl" scale="0.01 0.01 0.01"/>
         </geometry>
-        <material name="green">
-          <color rgba="0 1 0 1"/>
-        </material>
-      </visual>
-      <collision>
-        <origin xyz="0 0 0" rpy="0 0 0" />
-        <geometry>
-          <mesh filename="package://kortex_description/arms/gen3_lite/${dof}dof/meshes/MugCylinder.stl" scale="0.001 0.001 0.001"/>
-        </geometry>
-      </collision>
-    </link>
-    <joint name="cup_joint" type="fixed">
-      <parent link="${prefix}end_effector_link"/>
-      <child link="source_cup"/>
-      <origin xyz="0.0 0 0.12" rpy="-1.57 03.14 0"/>
-    </joint>
-    <link name="coffee_cup">
-      <visual>
-        <geometry>
-          <mesh filename="package://kortex_description/arms/gen3_lite/${dof}dof/meshes/papercup.stl" scale="1 1 1"/>
-        </geometry>
-        <material name="green">
-          <color rgba="0 1 0 1"/>
-        </material>
-      </visual>
-      <collision>
-        <origin xyz="0 0 0" rpy="0 0 0" />
-        <geometry>
-          <mesh filename="package://kortex_description/arms/gen3_lite/${dof}dof/meshes/papercup.stl" scale="0.001 0.001 0.001"/>
-        </geometry>
-      </collision>
-    </link>
-    <joint name="papercup_joint" type="fixed">
-      <parent link="${prefix}end_effector_link"/>
-      <child link="coffee_cup"/>
-      <origin xyz="0.0 0 0.12" rpy="-1.57 0 -1.57"/>
-    </joint>
-    <link name="soda_can">
-      <visual>
-        <geometry>
-          <mesh filename="package://kortex_description/arms/gen3_lite/${dof}dof/meshes/beverage_can.fbx" scale="0.01 0.01 0.01"/>
-        </geometry>
-        <material name="green">
-          <color rgba="0 1 0 1"/>
-        </material>
-      </visual>
-      <collision>
-        <origin xyz="0 0 0" rpy="0 0 0" />
-        <geometry>
-          <mesh filename="package://kortex_description/arms/gen3_lite/${dof}dof/meshes/beverage_can.fbx" scale="0.001 0.001 0.001"/>
-        </geometry>
-      </collision>
-    </link>
-    <joint name="sodacan_joint" type="fixed">
-      <parent link="${prefix}end_effector_link"/>
-      <child link="soda_can"/>
-      <origin xyz="-0.04 0.0 0.12" rpy="0 0 -1.57"/>
-    </joint>
-    <!-- <link name="beer_bottle">
-      <visual>
-        <geometry>
-          <mesh filename="package://kortex_description/arms/gen3_lite/${dof}dof/meshes/beer_bottle.stl" scale="0.001 0.001 0.001"/>
-        </geometry>
-        <material name="green">
-          <color rgba="0 1 0 1"/>
-        </material>
-      </visual>
-      <collision>
-        <origin xyz="0 0 0" rpy="0 0 0" />
-        <geometry>
-          <mesh filename="package://kortex_description/arms/gen3_lite/${dof}dof/meshes/beer_bottle.stl" scale="0.001 0.001 0.001"/>
-        </geometry>
-      </collision>
-    </link>
-    <joint name="waterbottle_joint" type="fixed">
-      <parent link="${prefix}end_effector_link"/>
-      <child link="beer_bottle"/>
-      <origin xyz="0.0 0.0 0.1" rpy="0 1.57 0"/>
-    </joint> -->
-    <link name="target_cup1">
-      <visual>
-        <origin xyz="0 0 0" rpy="0 0 0" />
-        <geometry>
-          <!-- <cylinder length="0.125" radius="0.0425"/> -->
-          <mesh filename="package://kortex_description/arms/gen3_lite/${dof}dof/meshes/MugCylinder.stl" scale="0.01 0.01 0.01"/>
-        </geometry>
         <material name="white">
           <color rgba="1 1 1 1"/>
@@ -123,5 +122,5 @@
     <joint name="cup_joint1" type="fixed">
       <parent link="table_link"/>
-      <child link="target_cup1"/>
+      <child link="Target_Cup"/>
       <origin xyz="0.0 -0.23 0.0625" rpy="0 1.57 0"/>
     </joint>
