Commit message: created new files for realsense2 camera integration

File: kortex_description/arms/gen3_lite/6dof/urdf/gen3_lite_macro_realsense2.xacro (robot description, xacro)
@@ -3,4 +3,16 @@
   <!-- Propagate last link name information because it is the gripper's parent link -->
   <xacro:property name="last_arm_link" value="dummy_link"/>
+  <!-- Intel RealSense D455 camera -->
+  <xacro:include filename="$(find realsense2_description)/urdf/_d455.urdf.xacro"/>
+  <xacro:sensor_d455 parent="camera_mount">
+    <origin xyz="0 0 0" rpy="0 0 0"/>
+  </xacro:sensor_d455>
+  <!-- Intel RealSense D455 camera -->
+  <link name="camera_mount"/>
+  <joint name="camera_to_frame" type="fixed">
+    <parent link="base_link"/>
+    <child link = "camera_mount"/>
+    <origin xyz="0 0 0" rpy="0 0 0"/>
+  </joint>
     <link name="table_link">
       <visual>
@@ -17,216 +29,4 @@
       <child link="table_link"/>
       <origin xyz="0.25 0 -0.05" rpy="0 0 1.57"/>
-    </joint>
-    <link name="01_Can">
-      <visual>
-        <geometry>
-          <mesh filename="package://kortex_description/arms/gen3_lite/${dof}dof/meshes/01_Can.stl" scale="0.01 0.01 0.01"/>
-        </geometry>
-        <material name="green">
-          <color rgba="0 1 0 1"/>
-        </material>
-      </visual>
-      <collision>
-        <origin xyz="0 0 0" rpy="0 0 0" />
-        <geometry>
-          <mesh filename="package://kortex_description/arms/gen3_lite/${dof}dof/meshes/01_Can.stl" scale="0.001 0.001 0.001"/>
-        </geometry>
-      </collision>
-    </link>
-    <joint name="can_joint" type="fixed">
-      <parent link="${prefix}end_effector_link"/>
-      <child link="01_Can"/>
-      <origin xyz="-0.045 0 0.108" rpy="-1.57 0 0"/>
-    </joint>
-    <link name="02_Wineglass">
-      <visual>
-        <geometry>
-          <mesh filename="package://kortex_description/arms/gen3_lite/${dof}dof/meshes/02_Wineglass.stl" scale="0.01 0.01 0.01"/>
-        </geometry>
-        <material name="green">
-          <color rgba="0 1 0 1"/>
-        </material>
-      </visual>
-      <collision>
-        <origin xyz="0 0 0" rpy="0 0 0" />
-        <geometry>
-          <mesh filename="package://kortex_description/arms/gen3_lite/${dof}dof/meshes/02_Wineglass.stl" scale="0.001 0.001 0.001"/>
-        </geometry>
-      </collision>
-    </link>
-    <joint name="wine_joint" type="fixed">
-      <parent link="${prefix}end_effector_link"/>
-      <child link="02_Wineglass"/>
-      <origin xyz="-0.026 0 0.105" rpy="-1.57 0 0"/>
-    </joint>
-    <link name="03_BlueCup">
-      <visual>
-        <geometry>
-          <mesh filename="package://kortex_description/arms/gen3_lite/${dof}dof/meshes/03_BlueCup.stl" scale="0.01 0.01 0.01"/>
-        </geometry>
-        <material name="green">
-          <color rgba="0 1 0 1"/>
-        </material>
-      </visual>
-      <collision>
-        <origin xyz="0 0 0" rpy="0 0 0" />
-        <geometry>
-          <mesh filename="package://kortex_description/arms/gen3_lite/${dof}dof/meshes/03_BlueCup.stl" scale="0.001 0.001 0.001"/>
-        </geometry>
-      </collision>
-    </link>
-    <joint name="blue_joint" type="fixed">
-      <parent link="${prefix}end_effector_link"/>
-      <child link="03_BlueCup"/>
-      <origin xyz="0.028 0 0.11" rpy="-1.57 0 0"/>
-    </joint>
-    <link name="04_plastic_water_bottle">
-      <visual>
-        <geometry>
-          <mesh filename="package://kortex_description/arms/gen3_lite/${dof}dof/meshes/04_plastic_water_bottle.stl" scale="0.01 0.01 0.01"/>
-        </geometry>
-        <material name="green">
-          <color rgba="0 1 0 1"/>
-        </material>
-      </visual>
-      <collision>
-        <origin xyz="0 0 0" rpy="0 0 0" />
-        <geometry>
-          <mesh filename="package://kortex_description/arms/gen3_lite/${dof}dof/meshes/04_plastic_water_bottle.stl" scale="0.0001 0.0001 0.0001"/>
-        </geometry>
-      </collision>
-    </link>
-    <joint name="plastic_joint" type="fixed">
-      <parent link="${prefix}end_effector_link"/>
-      <child link="04_plastic_water_bottle"/>
-      <origin xyz="0.028 0 0.11" rpy="-1.57 0 0"/>
-    </joint>
-    <link name="05_sports_bottle">
-      <visual>
-        <geometry>
-          <mesh filename="package://kortex_description/arms/gen3_lite/${dof}dof/meshes/05_sports_bottle.stl" scale="0.011 0.01 0.01"/>
-        </geometry>
-        <material name="green">
-          <color rgba="0 1 0 1"/>
-        </material>
-      </visual>
-      <collision>
-        <origin xyz="0 0 0" rpy="0 0 0" />
-        <geometry>
-          <mesh filename="package://kortex_description/arms/gen3_lite/${dof}dof/meshes/05_sports_bottle.stl" scale="0.0001 0.0001 0.0001"/>
-        </geometry>
-      </collision>
-    </link>
-    <joint name="sport_joint" type="fixed">
-      <parent link="${prefix}end_effector_link"/>
-      <child link="05_sports_bottle"/>
-      <origin xyz="-0.185 0 0.115" rpy="1.57 0 0"/>
-      <!-- <origin xyz="-0.155 0 0.115" rpy="1.57 0 0"/> -->
-    </joint>
-    <link name="06_tumbler">
-      <visual>
-        <geometry>
-          <mesh filename="package://kortex_description/arms/gen3_lite/${dof}dof/meshes/06_tumbler.stl" scale="0.01 0.01 0.01"/>
-        </geometry>
-        <material name="green">
-          <color rgba="0 1 0 1"/>
-        </material>
-      </visual>
-      <collision>
-        <origin xyz="0 0 0" rpy="0 0 0" />
-        <geometry>
-          <mesh filename="package://kortex_description/arms/gen3_lite/${dof}dof/meshes/06_tumbler.stl" scale="0.0001 0.0001 0.0001"/>
-        </geometry>
-      </collision>
-    </link>
-    <joint name="tumbler_joint" type="fixed">
-      <parent link="${prefix}end_effector_link"/>
-      <child link="06_tumbler"/>
-      <origin xyz="-0.155 0 0.12" rpy="1.57 0 0"/>
-    </joint>
-    <link name="07_Container">
-      <visual>
-        <geometry>
-          <mesh filename="package://kortex_description/arms/gen3_lite/${dof}dof/meshes/07_Container.stl" scale="0.01 0.01 0.01"/>
-        </geometry>
-        <material name="green">
-          <color rgba="0 1 0 1"/>
-        </material>
-      </visual>
-      <collision>
-        <origin xyz="0 0 0" rpy="0 0 0" />
-        <geometry>
-          <mesh filename="package://kortex_description/arms/gen3_lite/${dof}dof/meshes/07_Container.stl" scale="0.001 0.001 0.001"/>
-        </geometry>
-      </collision>
-    </link>
-    <joint name="container_joint" type="fixed">
-      <parent link="${prefix}end_effector_link"/>
-      <child link="07_Container"/>
-      <origin xyz="0.01 0 0.12" rpy="1.57 0 0"/>
-    </joint>
-    <link name="08_beerbottle">
-      <visual>
-        <geometry>
-          <mesh filename="package://kortex_description/arms/gen3_lite/${dof}dof/meshes/08_beerbottle.stl" scale="0.011 0.01 0.01"/>
-        </geometry>
-        <material name="green">
-          <color rgba="0 1 0 1"/>
-        </material>
-      </visual>
-      <collision>
-        <origin xyz="0 0 0" rpy="0 0 0" />
-        <geometry>
-          <mesh filename="package://kortex_description/arms/gen3_lite/${dof}dof/meshes/08_beerbottle.stl" scale="0.0001 0.0001 0.0001"/>
-        </geometry>
-      </collision>
-    </link>
-    <joint name="rootbeer_joint" type="fixed">
-      <parent link="${prefix}end_effector_link"/>
-      <child link="08_beerbottle"/>
-      <!-- <origin xyz="-0.07 0 0.105" rpy="1.57 0 0"/> -->
-      <origin xyz="-0.08 0 0.105" rpy="1.57 0 0"/>
-    </joint>
-    <link name="09_Paper_cup">
-      <visual>
-        <geometry>
-          <mesh filename="package://kortex_description/arms/gen3_lite/${dof}dof/meshes/09_Paper_cup.stl" scale="0.01 0.01 0.01"/>
-        </geometry>
-        <material name="green">
-          <color rgba="0 1 0 1"/>
-        </material>
-      </visual>
-      <collision>
-        <origin xyz="0 0 0" rpy="0 0 0" />
-        <geometry>
-          <mesh filename="package://kortex_description/arms/gen3_lite/${dof}dof/meshes/09_Paper_cup.stl" scale="0.001 0.001 0.001"/>
-        </geometry>
-      </collision>
-    </link>
-    <joint name="paper_joint" type="fixed">
-      <parent link="${prefix}end_effector_link"/>
-      <child link="09_Paper_cup"/>
-      <origin xyz="0.03 0 0.11" rpy="1.57 0 0"/>
-    </joint>
-    <link name="10_mug">
-      <visual>
-        <geometry>
-          <mesh filename="package://kortex_description/arms/gen3_lite/${dof}dof/meshes/10_mug.stl" scale="0.011 0.01 0.01"/>
-        </geometry>
-        <material name="green">
-          <color rgba="0 1 0 1"/>
-        </material>
-      </visual>
-      <collision>
-        <origin xyz="10 0 0" rpy="0 0 0" />
-        <geometry>
-          <mesh filename="package://kortex_description/arms/gen3_lite/${dof}dof/meshes/10_mug.stl" scale="0.001 0.001 0.001"/>
-        </geometry>
-      </collision>
-    </link>
-    <joint name="mug_joint" type="fixed">
-      <parent link="${prefix}end_effector_link"/>
-      <child link="10_mug"/>
-      <origin xyz="-0.04 0 0.12" rpy="1.57 0 0"/>
     </joint>
     <link name="Target_Cup">
